Commit message: Added rotary offset. Also added markers to cylinder.

File: multibody/models/cylinder_flat.urdf (robot description, URDF)
Before this commit: robot cylinder, 1 links, 0 joints
Links:
- link cylinder: geometry collision cylinder length=0.04 radius=0.03; visual cylinder length=0.04 radius=0.03
